File: CyborgHD6309E/Prototype5/schematic/Prototype5.kicad_pcb (KiCad board)
At the start: 2 copper layers, 95 x 72 mm, 22 parts, among them J1 Conn_AVR_UPDI, SW1 TSD1265, U1 ATmega4809-P, U2 HM628128DLP-5, U3 HD63C09E, U5 CD74HCT30, U6 CD74HCT688

Commit message: [CyborgHD6309E] Prorotype5 debugger
Parts:
- removed C5: 0.1u, Capacitor_THT:C_Disc_D3.4mm_W2.1mm_P2.50mm
- removed U5: CD74HCT30, Package_DIP:DIP-14_W7.62mm
- added RN1: 100k, Resistor_THT:R_Array_SIP9, F.Cu at (102.3, 105.6)
- added SW2: SW_DIP_x08, Package_DIP:DIP-16_W7.62mm, F.Cu at (106.1, 108.1)
- moved R2 5.08 mm to (164.5, 110.6), turned to 270 degrees
- moved C6 2.54 mm to (102.3, 77.6)
Connections:
- U1 pad 25: /~IOR~ -> /E_CLK
- U1 pad 26: /E_CLK -> /~IOR~
- U1 pad 3: /~RAM_E~ -> /Q_CLK
- U1 pad 4: /Q_CLK -> /~RAM_E~
- U2 pad 10: /A10 -> /A2
- U2 pad 11: /A11 -> /A1
- U2 pad 12: /A12 -> /A0
- U2 pad 13: /D5 -> /D0
- U2 pad 14: /D6 -> /D1
- U2 pad 15: /D7 -> /D2
- U2 pad 17: /D4 -> /D3
- U2 pad 18: /D3 -> /D4
- U2 pad 19: /D2 -> /D5
- U2 pad 20: /D1 -> /D6
- U2 pad 21: /D0 -> /D7
- U2 pad 23: /A2 -> /A10
- U2 pad 25: /A1 -> /A11
- U2 pad 26: /A0 -> /A9
- U2 pad 27: /A13 -> /A8
- U2 pad 28: /A14 -> /A13
- U2 pad 3: /A3 -> /A14
- U2 pad 4: /A4 -> /A12
- U2 pad 5: /A5 -> /A7
- U2 pad 7: /A7 -> /A5
- U2 pad 8: /A8 -> /A4
- U2 pad 9: /A9 -> /A3
- U3 pad 34: /Q_CLK -> /E_CLK
- U3 pad 35: /E_CLK -> /Q_CLK
- U6 pad 1: Net-(U5-Pad8) -> GND
- U6 pad 11: /A6 -> /A12
- U6 pad 12: VCC -> Net-(RN1-Pad6)
- U6 pad 13: /A5 -> /A13
- U6 pad 14: GND -> Net-(RN1-Pad7)
- U6 pad 15: /A4 -> /A14
- U6 pad 16: GND -> Net-(RN1-Pad8)
- U6 pad 17: /A3 -> /A15
- U6 pad 18: GND -> Net-(RN1-Pad9)
- U6 pad 2: GND -> /A8
- U6 pad 3: GND -> Net-(RN1-Pad2)
- U6 pad 4: GND -> /A9
- U6 pad 5: GND -> Net-(RN1-Pad3)
- U6 pad 6: GND -> /A10
- U6 pad 7: GND -> Net-(RN1-Pad4)
- U6 pad 8: /A7 -> /A11
- U6 pad 9: VCC -> Net-(RN1-Pad5)
